File: hardware/KiCad/UVK5_reversing_06-02-2024/Charger.kicad_sch (KiCad schematic)
At the start: 18 parts, among them J27 Batt-Con +, J28 Batt-Con -, Q30 2TY, S8550, Q31 D882, T21 Transformer_SP_1S, U23 TL431D

Commit message: 14.08.2025
Parts:
- removed C92: 470µF 16V, symbol UV-K5:C
- removed D42: Green_LED, symbol UV-K5:LED
- removed T21: Transformer_SP_1S, symbol UV-K5:Transformer_SP_1S
- added C1: 4,7 µF 400 V, symbol Device:C_Polarized
- added C2: ~, symbol UV-K5:C
- added C3: 470 µF 16 V, symbol Device:C_Polarized
- added C4: ? 50V, symbol UV-K5:C
- added C5: 4,7 µF 50 V, symbol Device:C_Polarized
- added D1: MB10F, Package_SO:OnSemi_751EP_SOIC-4_3.9x4.725mm_P2.54mm, symbol Diode_Bridge:MB8S
- added D2, D3: A7, symbol Device:D
- added D4: Green_LED, symbol UV-K5:LED
- added J1: L, symbol UV-K5:Conn_01x01_Pin
- added J2: N, symbol UV-K5:Conn_01x01_Pin
- added R2: 200k, symbol UV-K5:R
- added R3: 2M2, symbol UV-K5:R
- added R4: 18k, symbol UV-K5:R
- added R5: 3K48, symbol UV-K5:R
- added R6: 330k, symbol UV-K5:R
- added TR1: ~, symbol Transformer:TRANSF3
- added U1: LP3783A, Package_TO_SOT_SMD:SOT-23-6, symbol Regulator_SwitchedCapacitor:LP3783A
- added r1: 1R8, symbol UV-K5:R
- D?: renamed from D43; value D -> K110
- R?: renamed from R56; value 2k2 -> 2,37K (1%)
- r?: renamed from r54; value 1K0 -> 1K
- renumbered C91 to C?, D41 to D?, J28 to J?, J27 to J?, Q31 to Q?, Q30 to Q?, R52 to R?, R57 to R?, R55 to R?, R53 to R?, R58 to R?, U23 to U?
Connections:
- net GND: now also C3.2, TR1.1
- net V+: now also C3.1, D4.2 (A)
- net at C?.1, J?.1 (Pin_1), Q?.3 (E)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: now also R6.1
- net at D?.1 (K), R?.1: now also D4.1 (K)
- net at R?.1, R?.2, U?.8 (REF): now also R6.2
- net at D?.2 (A): now also TR1.2
- new net: D1.3, J1.1 (Pin_1)
- new net: R4.1, R5.2, U1.1 (FB)
- new net: U1.2 (CS), U1.4 (E), r1.1
- new net: C4.1, C5.1, D2.1 (K), R3.1, U1.3 (VCC)
- new net: D3.2 (A), TR1.5, U1.5 (C), U1.6 (C)
- new net: D2.2 (A), R4.2, TR1.4
- new net: D1.4, J2.1 (Pin_1)
- new net: C1.1, C2.1, D1.1 (+), R2.1, R3.2, TR1.6
- new net: C2.2, D3.1 (K), R2.2
- new net GNDPWR: C1.2, C4.2, C5.2, D1.2 (-), R5.1, TR1.3, U1.7 (GND), r1.2
Other:
- note added: "2 x 4,2 V"
- note added: "Batt-Conn + 8,4V without Load"
- note added: "Origin Postet By Tom George Corrected by Matteo Portet to KiCad by Ludwich Completed by Daniel Eastwood 08/2025"
- note removed: "Origin Postet By Tom George Corrected by Matteo Portet to KiCad by Ludwich"
- note removed: "V+ 9,7 V without Load Batt-Conn + 8,3V without Load"
- moved on the sheet: C?
